File: tung_40/tung_40.kicad_pcb (KiCad board)
At the start: 2 copper layers, 7 parts, among them J1 Conn_01x02_Male, J2 Conn_01x02_Male, SW1 GateronLP, SW5 SW_DIP_x03, U1 NRF52840-DONGLE

Commit message: 48 keys in progress
Parts:
- removed D1: 1N4148, Diode_THT:D_DO-35_SOD27_P7.62mm_Horizontal
- removed J2: Conn_01x02_Male, Connector_PinHeader_2.54mm:PinHeader_1x02_P2.54mm_Vertical
- removed SW1: GateronLP, Button_Switch_Keyboard:SW_Cherry_MX_1.00u_PCB
- added D11: 1N4148, Diode_THT:D_DO-35_SOD27_P7.62mm_Horizontal, F.Cu at (-9.53, 9.53)
- added D110: 1N4148, Diode_THT:D_DO-35_SOD27_P7.62mm_Horizontal, F.Cu at (-4.76, 19.1)
- added D12: 1N4148, Diode_THT:D_DO-35_SOD27_P7.62mm_Horizontal, F.Cu at (-23.8, 9.53)
- added D13: 1N4148, Diode_THT:D_DO-35_SOD27_P7.62mm_Horizontal, F.Cu at (-38.1, 4.76)
- added D14: 1N4148, Diode_THT:D_DO-35_SOD27_P7.62mm_Horizontal, F.Cu at (-28.6, 0.00)
- added D15: 1N4148, Diode_THT:D_DO-35_SOD27_P7.62mm_Horizontal, F.Cu at (-15.5, 0.00)
- added D16: 1N4148, Diode_THT:D_DO-35_SOD27_P7.62mm_Horizontal, F.Cu at (-47.6, 9.53)
- added D17: 1N4148, Diode_THT:D_DO-35_SOD27_P7.62mm_Horizontal, F.Cu at (-38.1, 14.3)
- added D18: 1N4148, Diode_THT:D_DO-35_SOD27_P7.62mm_Horizontal, F.Cu at (-19.1, 14.3)
- added D19: 1N4148, Diode_THT:D_DO-35_SOD27_P7.62mm_Horizontal, F.Cu at (-23.8, 4.76)
- added D21: 1N4148, Diode_THT:D_DO-35_SOD27_P7.62mm_Horizontal, F.Cu at (-14.3, 33.3)
- added D210: 1N4148, Diode_THT:D_DO-35_SOD27_P7.62mm_Horizontal, F.Cu at (-26.6, 40.4)
- added D22: 1N4148, Diode_THT:D_DO-35_SOD27_P7.62mm_Horizontal, F.Cu at (-38.1, 33.3)
- added D23: 1N4148, Diode_THT:D_DO-35_SOD27_P7.62mm_Horizontal, F.Cu at (-38.1, 27.3)
- added D24: 1N4148, Diode_THT:D_DO-35_SOD27_P7.62mm_Horizontal, F.Cu at (-28.6, 23.8)
- added D25: 1N4148, Diode_THT:D_DO-35_SOD27_P7.62mm_Horizontal, F.Cu at (-9.53, 28.6)
- added D26: 1N4148, Diode_THT:D_DO-35_SOD27_P7.62mm_Horizontal, F.Cu at (-14.3, 38.1)
- added D27: 1N4148, Diode_THT:D_DO-35_SOD27_P7.62mm_Horizontal, F.Cu at (-23.8, 28.6)
- added D28: 1N4148, Diode_THT:D_DO-35_SOD27_P7.62mm_Horizontal, F.Cu at (-38.1, 38.1)
- added D29: 1N4148, Diode_THT:D_DO-35_SOD27_P7.62mm_Horizontal, F.Cu at (-23.8, 33.3)
- added D31: 1N4148, Diode_THT:D_DO-35_SOD27_P7.62mm_Horizontal, F.Cu at (-4.76, 52.4)
- added D310: 1N4148, Diode_THT:D_DO-35_SOD27_P7.62mm_Horizontal, F.Cu at (-4.76, 57.1)
- added D32: 1N4148, Diode_THT:D_DO-35_SOD27_P7.62mm_Horizontal, F.Cu at (-13.4, 58.4)
- added D33: 1N4148, Diode_THT:D_DO-35_SOD27_P7.62mm_Horizontal, F.Cu at (-15.5, 64.3)
- added D34: 1N4148, Diode_THT:D_DO-35_SOD27_P7.62mm_Horizontal, F.Cu at (-15.5, 67.9)
- added D35: 1N4148, Diode_THT:D_DO-35_SOD27_P7.62mm_Horizontal, F.Cu at (-14.3, 52.4)
- added D36: 1N4148, Diode_THT:D_DO-35_SOD27_P7.62mm_Horizontal, F.Cu at (-4.76, 64.3)
- added D37: 1N4148, Diode_THT:D_DO-35_SOD27_P7.62mm_Horizontal, F.Cu at (-4.76, 71.4)
- added D38: 1N4148, Diode_THT:D_DO-35_SOD27_P7.62mm_Horizontal, F.Cu at (-9.53, 47.6)
- added D39: 1N4148, Diode_THT:D_DO-35_SOD27_P7.62mm_Horizontal, F.Cu at (-23.8, 47.6)
- added D41: 1N4148, Diode_THT:D_DO-35_SOD27_P7.62mm_Horizontal, F.Cu at (-71.4, 38.1)
- added D410: 1N4148, Diode_THT:D_DO-35_SOD27_P7.62mm_Horizontal, F.Cu at (-61.9, 52.4)
- added D42: 1N4148, Diode_THT:D_DO-35_SOD27_P7.62mm_Horizontal, F.Cu at (-66.7, 42.9)
- added D43: 1N4148, Diode_THT:D_DO-35_SOD27_P7.62mm_Horizontal, F.Cu at (-52.4, 44.1)
- added D44: 1N4148, Diode_THT:D_DO-35_SOD27_P7.62mm_Horizontal, F.Cu at (-50.3, 52.4)
- added D45: 1N4148, Diode_THT:D_DO-35_SOD27_P7.62mm_Horizontal, F.Cu at (-66.7, 29.8)
- added D46: 1N4148, Diode_THT:D_DO-35_SOD27_P7.62mm_Horizontal, F.Cu at (-66.7, 33.3)
- added D47: 1N4148, Diode_THT:D_DO-35_SOD27_P7.62mm_Horizontal, F.Cu at (-55.5, 38.1)
- added D48: 1N4148, Diode_THT:D_DO-35_SOD27_P7.62mm_Horizontal, F.Cu at (-61.9, 47.6)
- added D49: 1N4148, Diode_THT:D_DO-35_SOD27_P7.62mm_Horizontal, F.Cu at (-52.4, 47.6)
- added D51: 1N4148, Diode_THT:D_DO-35_SOD27_P7.62mm_Horizontal, F.Cu at (-47.6, 61.9)
- added D52: 1N4148, Diode_THT:D_DO-35_SOD27_P7.62mm_Horizontal, F.Cu at (-52.4, 75.0)
- added D53: 1N4148, Diode_THT:D_DO-35_SOD27_P7.62mm_Horizontal, F.Cu at (-42.9, 71.4)
- added D54: 1N4148, Diode_THT:D_DO-35_SOD27_P7.62mm_Horizontal, F.Cu at (-27.5, 70.2)
- added D55: 1N4148, Diode_THT:D_DO-35_SOD27_P7.62mm_Horizontal, F.Cu at (-28.6, 71.4)
- added D56: 1N4148, Diode_THT:D_DO-35_SOD27_P7.62mm_Horizontal, F.Cu at (-33.3, 61.9)
- added D57: 1N4148, Diode_THT:D_DO-35_SOD27_P7.62mm_Horizontal, F.Cu at (-42.9, 66.7)
- added D58: 1N4148, Diode_THT:D_DO-35_SOD27_P7.62mm_Horizontal, F.Cu at (-38.1, 76.2)
- added SW11: GateronLP, GateronLP:SW_Gateron_LO_PRO_1.00u_NO_LED_REVERSABLE_PCB, F.Cu at (14.3, 14.3)
- added SW110: GateronLP, GateronLP:SW_Gateron_LO_PRO_1.00u_NO_LED_REVERSABLE_PCB, F.Cu at (261.9, 14.3)
- added SW12: GateronLP, GateronLP:SW_Gateron_LO_PRO_1.00u_NO_LED_REVERSABLE_PCB, F.Cu at (33.3, 14.3)
- added SW13: GateronLP, GateronLP:SW_Gateron_LO_PRO_1.00u_NO_LED_REVERSABLE_PCB, F.Cu at (52.4, 14.3)
- added SW14: GateronLP, GateronLP:SW_Gateron_LO_PRO_1.00u_NO_LED_REVERSABLE_PCB, F.Cu at (71.4, 14.3)
- added SW15: GateronLP, GateronLP:SW_Gateron_LO_PRO_1.00u_NO_LED_REVERSABLE_PCB, F.Cu at (90.5, 14.3)
- added SW16: GateronLP, GateronLP:SW_Gateron_LO_PRO_1.00u_NO_LED_REVERSABLE_PCB, F.Cu at (185.7, 14.3)
- added SW17: GateronLP, GateronLP:SW_Gateron_LO_PRO_1.00u_NO_LED_REVERSABLE_PCB, F.Cu at (204.8, 14.3)
- added SW18: GateronLP, GateronLP:SW_Gateron_LO_PRO_1.00u_NO_LED_REVERSABLE_PCB, F.Cu at (223.8, 14.3)
- added SW19: GateronLP, GateronLP:SW_Gateron_LO_PRO_1.00u_NO_LED_REVERSABLE_PCB, F.Cu at (242.9, 14.3)
- added SW21: GateronLP, GateronLP:SW_Gateron_LO_PRO_1.00u_NO_LED_REVERSABLE_PCB, F.Cu at (14.3, 33.3)
- added SW210: GateronLP, GateronLP:SW_Gateron_LO_PRO_1.00u_NO_LED_REVERSABLE_PCB, F.Cu at (261.9, 33.3)
- added SW22: GateronLP, GateronLP:SW_Gateron_LO_PRO_1.00u_NO_LED_REVERSABLE_PCB, F.Cu at (33.3, 33.3)
- added SW23: GateronLP, GateronLP:SW_Gateron_LO_PRO_1.00u_NO_LED_REVERSABLE_PCB, F.Cu at (52.4, 33.3)
- added SW24: GateronLP, GateronLP:SW_Gateron_LO_PRO_1.00u_NO_LED_REVERSABLE_PCB, F.Cu at (71.4, 33.3)
- added SW25: GateronLP, GateronLP:SW_Gateron_LO_PRO_1.00u_NO_LED_REVERSABLE_PCB, F.Cu at (90.5, 33.3)
- added SW26: GateronLP, GateronLP:SW_Gateron_LO_PRO_1.00u_NO_LED_REVERSABLE_PCB, F.Cu at (185.7, 33.3)
- added SW27: GateronLP, GateronLP:SW_Gateron_LO_PRO_1.00u_NO_LED_REVERSABLE_PCB, F.Cu at (204.8, 33.3)
- added SW28: GateronLP, GateronLP:SW_Gateron_LO_PRO_1.00u_NO_LED_REVERSABLE_PCB, F.Cu at (223.8, 33.3)
- added SW29: GateronLP, GateronLP:SW_Gateron_LO_PRO_1.00u_NO_LED_REVERSABLE_PCB, F.Cu at (242.9, 33.3)
- added SW31: GateronLP, GateronLP:SW_Gateron_LO_PRO_1.00u_NO_LED_REVERSABLE_PCB, F.Cu at (14.3, 52.4)
- added SW310: GateronLP, GateronLP:SW_Gateron_LO_PRO_1.00u_NO_LED_REVERSABLE_PCB, F.Cu at (261.9, 52.4)
- added SW32: GateronLP, GateronLP:SW_Gateron_LO_PRO_1.00u_NO_LED_REVERSABLE_PCB, F.Cu at (33.3, 52.4)
- added SW33: GateronLP, GateronLP:SW_Gateron_LO_PRO_1.00u_NO_LED_REVERSABLE_PCB, F.Cu at (52.4, 52.4)
- added SW34: GateronLP, GateronLP:SW_Gateron_LO_PRO_1.00u_NO_LED_REVERSABLE_PCB, F.Cu at (71.4, 52.4)
- added SW35: GateronLP, GateronLP:SW_Gateron_LO_PRO_1.00u_NO_LED_REVERSABLE_PCB, F.Cu at (90.5, 52.4)
- added SW36: GateronLP, GateronLP:SW_Gateron_LO_PRO_1.00u_NO_LED_REVERSABLE_PCB, F.Cu at (185.7, 52.4)
- added SW37: GateronLP, GateronLP:SW_Gateron_LO_PRO_1.00u_NO_LED_REVERSABLE_PCB, F.Cu at (204.8, 52.4)
- added SW38: GateronLP, GateronLP:SW_Gateron_LO_PRO_1.00u_NO_LED_REVERSABLE_PCB, F.Cu at (223.8, 52.4)
- added SW39: GateronLP, GateronLP:SW_Gateron_LO_PRO_1.00u_NO_LED_REVERSABLE_PCB, F.Cu at (242.9, 52.4)
- added SW41: GateronLP, GateronLP:SW_Gateron_LO_PRO_1.00u_NO_LED_REVERSABLE_PCB, F.Cu at (14.3, 71.4)
- added SW410: GateronLP, GateronLP:SW_Gateron_LO_PRO_1.00u_NO_LED_REVERSABLE_PCB, F.Cu at (261.9, 71.4)
- added SW42: GateronLP, GateronLP:SW_Gateron_LO_PRO_1.00u_NO_LED_REVERSABLE_PCB, F.Cu at (33.3, 71.4)
- added SW43: GateronLP, GateronLP:SW_Gateron_LO_PRO_1.00u_NO_LED_REVERSABLE_PCB, F.Cu at (52.4, 71.4)
- added SW44: GateronLP, GateronLP:SW_Gateron_LO_PRO_1.00u_NO_LED_REVERSABLE_PCB, F.Cu at (71.4, 71.4)
- added SW45: GateronLP, GateronLP:SW_Gateron_LO_PRO_1.00u_NO_LED_REVERSABLE_PCB, F.Cu at (90.5, 71.4)
- added SW46: GateronLP, GateronLP:SW_Gateron_LO_PRO_1.00u_NO_LED_REVERSABLE_PCB, F.Cu at (185.7, 71.4)
- added SW47: GateronLP, GateronLP:SW_Gateron_LO_PRO_1.00u_NO_LED_REVERSABLE_PCB, F.Cu at (204.8, 71.4)
- added SW48: GateronLP, GateronLP:SW_Gateron_LO_PRO_1.00u_NO_LED_REVERSABLE_PCB, F.Cu at (223.8, 71.4)
- added SW49: GateronLP, GateronLP:SW_Gateron_LO_PRO_1.00u_NO_LED_REVERSABLE_PCB, F.Cu at (242.9, 71.4)
- added SW51: GateronLP, GateronLP:SW_Gateron_LO_PRO_1.00u_NO_LED_REVERSABLE_PCB, F.Cu at (109.5, 14.3)
- added SW52: GateronLP, GateronLP:SW_Gateron_LO_PRO_1.00u_NO_LED_REVERSABLE_PCB, F.Cu at (109.5, 33.3)
- added SW53: GateronLP, GateronLP:SW_Gateron_LO_PRO_1.00u_NO_LED_REVERSABLE_PCB, F.Cu at (109.5, 52.4)
- added SW54: GateronLP, GateronLP:SW_Gateron_LO_PRO_1.00u_NO_LED_REVERSABLE_PCB, F.Cu at (109.5, 71.4)
- added SW55: GateronLP, GateronLP:SW_Gateron_LO_PRO_1.00u_NO_LED_REVERSABLE_PCB, F.Cu at (166.7, 71.4)
- added SW56: GateronLP, GateronLP:SW_Gateron_LO_PRO_1.00u_NO_LED_REVERSABLE_PCB, F.Cu at (166.7, 52.4)
- added SW57: GateronLP, GateronLP:SW_Gateron_LO_PRO_1.00u_NO_LED_REVERSABLE_PCB, F.Cu at (166.7, 33.3)
- added SW58: GateronLP, GateronLP:SW_Gateron_LO_PRO_1.00u_NO_LED_REVERSABLE_PCB, F.Cu at (166.7, 14.3)
- BT1: footprint Battery:Battery_Panasonic_CR2032-VS1N_Vertical_CircularHoles -> Misc:TBH-CR2032-M04
- SW5: value SW_DIP_x03 -> SW_DIP_x02; footprint Button_Switch_THT:SW_DIP_SPSTx02_Slide_6.7x6.64mm_W7.62mm_P2.54mm_LowProfile -> Misc:SW_DIP_SPSTx02_Slide_9.78x7.26mm_W7.62mm_P2.54mm
- moved BT1 437.9 mm to (138.1, 71.4), turned to 180 degrees
- moved U1 424.4 mm to (138.1, 28.6), turned to 90 degrees
- moved SW5 399.1 mm to (95.2, -19.1), turned to 180 degrees
- moved J1 212.8 mm to (-61.9, 66.7), turned to 180 degrees
Connections:
- U1 pad 0.02: unconnected-(U1-Pad0.02) -> Net-(SW11-Pad1)
- U1 pad 0.09: unconnected-(U1-Pad0.09) -> Net-(SW12-Pad1)
- U1 pad 0.10: unconnected-(U1-Pad0.10) -> Net-(D11-Pad1)
- U1 pad 0.13: unconnected-(U1-Pad0.13) -> Net-(D21-Pad1)
- U1 pad 0.15: unconnected-(U1-Pad0.15) -> Net-(D39-Pad1)
- U1 pad 0.17: unconnected-(U1-Pad0.17) -> Net-(D49-Pad1)
- U1 pad 0.20: unconnected-(U1-Pad0.20) -> Net-(D57-Pad1)
- U1 pad 0.22: unconnected-(U1-Pad0.22) -> Net-(SW13-Pad1)
- U1 pad 0.24: unconnected-(U1-Pad0.24) -> Net-(SW14-Pad1)
- U1 pad 0.29: unconnected-(U1-Pad0.29) -> Net-(SW15-Pad1)
- U1 pad 0.31: unconnected-(U1-Pad0.31) -> Net-(SW16-Pad1)
- U1 pad 1.00: unconnected-(U1-Pad1.00) -> Net-(SW17-Pad1)
- U1 pad 1.10: unconnected-(U1-Pad1.10) -> Net-(SW18-Pad1)
- U1 pad 1.13: unconnected-(U1-Pad1.13) -> Net-(SW39-Pad1)
- U1 pad 1.15: unconnected-(U1-Pad1.15) -> Net-(SW110-Pad1)

Commit message: continue 48 keys
Parts:
- moved D410 315.2 mm to (252.4, 75.4), turned to 90 degrees
- moved D49 287.1 mm to (233.4, 75.4), turned to 90 degrees
- moved D210 279.0 mm to (252.4, 37.3), turned to 90 degrees
- moved D48 277.6 mm to (214.3, 75.4), turned to 90 degrees
- moved D19 257.5 mm to (233.4, 18.2), turned to 90 degrees
- moved D39 257.3 mm to (233.4, 56.3), turned to 90 degrees
- moved D29 257.2 mm to (233.4, 37.3), turned to 90 degrees
- moved D110 257.2 mm to (252.4, 18.2), turned to 90 degrees
- moved D310 257.2 mm to (252.4, 56.3), turned to 90 degrees
- moved D47 253.6 mm to (195.3, 75.4), turned to 90 degrees
- moved D28 252.4 mm to (214.3, 37.3), turned to 90 degrees
- moved D46 246.5 mm to (176.2, 75.4), turned to 90 degrees
- moved D18 233.4 mm to (214.3, 18.2), turned to 90 degrees
- moved D17 233.4 mm to (195.3, 18.2), turned to 90 degrees
- moved D16 224.0 mm to (176.2, 18.2), turned to 90 degrees
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Connections:
- D31 pad 1: Net-(D39-Pad1) -> Net-(D31-Pad1)
- D310 pad 1: Net-(D39-Pad1) -> Net-(D31-Pad1)
- D32 pad 1: Net-(D39-Pad1) -> Net-(D31-Pad1)
- D33 pad 1: Net-(D39-Pad1) -> Net-(D31-Pad1)
- D34 pad 1: Net-(D39-Pad1) -> Net-(D31-Pad1)
- D35 pad 1: Net-(D39-Pad1) -> Net-(D31-Pad1)
- D36 pad 1: Net-(D39-Pad1) -> Net-(D31-Pad1)
- D37 pad 1: Net-(D39-Pad1) -> Net-(D31-Pad1)
- D38 pad 1: Net-(D39-Pad1) -> Net-(D31-Pad1)
- D39 pad 1: Net-(D39-Pad1) -> Net-(D31-Pad1)
- D41 pad 1: Net-(D49-Pad1) -> Net-(D41-Pad1)
- D410 pad 1: Net-(D49-Pad1) -> Net-(D41-Pad1)
- D42 pad 1: Net-(D49-Pad1) -> Net-(D41-Pad1)
- D43 pad 1: Net-(D49-Pad1) -> Net-(D41-Pad1)
- D44 pad 1: Net-(D49-Pad1) -> Net-(D41-Pad1)
- D45 pad 1: Net-(D49-Pad1) -> Net-(D41-Pad1)
- D46 pad 1: Net-(D49-Pad1) -> Net-(D41-Pad1)
- D47 pad 1: Net-(D49-Pad1) -> Net-(D41-Pad1)
- D48 pad 1: Net-(D49-Pad1) -> Net-(D41-Pad1)
- D49 pad 1: Net-(D49-Pad1) -> Net-(D41-Pad1)
- D51 pad 1: Net-(D57-Pad1) -> Net-(D51-Pad1)
- D52 pad 1: Net-(D57-Pad1) -> Net-(D51-Pad1)
- D53 pad 1: Net-(D57-Pad1) -> Net-(D51-Pad1)
- D54 pad 1: Net-(D57-Pad1) -> Net-(D51-Pad1)
- D55 pad 1: Net-(D57-Pad1) -> Net-(D51-Pad1)
- D56 pad 1: Net-(D57-Pad1) -> Net-(D51-Pad1)
- D57 pad 1: Net-(D57-Pad1) -> Net-(D51-Pad1)
- D58 pad 1: Net-(D57-Pad1) -> Net-(D51-Pad1)
- SW19 pad 1: Net-(SW39-Pad1) -> Net-(SW19-Pad1)
- SW29 pad 1: Net-(SW39-Pad1) -> Net-(SW19-Pad1)
- SW39 pad 1: Net-(SW39-Pad1) -> Net-(SW19-Pad1)
- SW49 pad 1: Net-(SW39-Pad1) -> Net-(SW19-Pad1)
- U1 pad 0.02: Net-(SW11-Pad1) -> unconnected-(U1-Pad0.02)
- U1 pad 0.09: Net-(SW12-Pad1) -> unconnected-(U1-Pad0.09)
- U1 pad 0.10: Net-(D11-Pad1) -> unconnected-(U1-Pad0.10)
- U1 pad 0.13: Net-(D21-Pad1) -> Net-(SW11-Pad1)
- U1 pad 0.15: Net-(D39-Pad1) -> Net-(SW12-Pad1)
- U1 pad 0.17: Net-(D49-Pad1) -> unconnected-(U1-Pad0.17)
- U1 pad 0.20: Net-(D57-Pad1) -> unconnected-(U1-Pad0.20)
- U1 pad 0.22: Net-(SW13-Pad1) -> unconnected-(U1-Pad0.22)
- U1 pad 0.24: Net-(SW14-Pad1) -> unconnected-(U1-Pad0.24)
- U1 pad 0.29: Net-(SW15-Pad1) -> unconnected-(U1-Pad0.29)
- U1 pad 0.31: Net-(SW16-Pad1) -> unconnected-(U1-Pad0.31)
- U1 pad 1.00: Net-(SW17-Pad1) -> unconnected-(U1-Pad1.00)
- U1 pad 1.10: Net-(SW18-Pad1) -> unconnected-(U1-Pad1.10)
- U1 pad 1.13: Net-(SW39-Pad1) -> unconnected-(U1-Pad1.13)
- U1 pad 1.15: Net-(SW110-Pad1) -> unconnected-(U1-Pad1.15)
Routing:
- net Net-(D21-Pad1): track 0.00 -> 263.7 mm
- net Net-(D11-Pad1): track 0.00 -> 235.2 mm
- net Net-(D41-Pad1): track 0.00 -> 230.2 mm
- net Net-(D31-Pad1): track 0.00 -> 229.8 mm
- net Net-(SW11-Pad1): track 0.00 -> 225.0 mm
- net Net-(SW12-Pad1): track 0.00 -> 192.8 mm
- net Net-(D51-Pad1): track 0.00 -> 173.3 mm
- net Net-(SW18-Pad1): track 0.00 -> 155.5 mm
- net Net-(SW13-Pad1): track 0.00 -> 153.4 mm
- net Net-(SW17-Pad1): track 0.00 -> 134.8 mm
- net Net-(SW14-Pad1): track 0.00 -> 134.6 mm
- net Net-(SW15-Pad1): track 0.00 -> 103.1 mm
- net Net-(SW16-Pad1): track 0.00 -> 100.9 mm
- net Net-(SW19-Pad1): track 0.00 -> 97.9 mm
- net Net-(SW110-Pad1): track 0.00 -> 96.8 mm
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